Commit message: fixed leg joints issues

File: urdf_drone/drone_ufo_v1.urdf (robot description, URDF)
Before this commit: robot triphibious_drone, 14 links, 13 joints
Joints:
- joint leg_1_joint: axis 0 0 -1 -> 0 0 1
- joint leg_2_joint: axis 0 0 -1 -> 0 0 1
- joint leg_3_joint: axis 0 0 -1 -> 0 0 1
- joint leg_4_joint: axis 0 0 -1 -> 0 0 1
- joint sphere_joint: limit (none) -> effort=2.0 velocity=3.0
